File: kicad/4N35-TTL-Serial-Optoisolator.sch (KiCad schematic (older format))
At the start: 12 parts, among them P1 CONN_4, P2 CONN_4, Q1 2N3906, Q2 2N3906, U1 4N35, U2 4N35

Commit message: v1
Other:
- note removed: "TODO: add capacitors? or is that only needed for 6N137?"
Changed lines of the file:
@@
 LIBS:contrib
 LIBS:valves
+LIBS:4N35-TTL-Serial-Optoisolator-cache
 EELAYER 27 0
 EELAYER END
@@
 	-1   0    0    -1
 $EndComp
-Text Notes 2450 5750 0    60   ~ 0
-TODO: add capacitors?  or is that only needed for 6N137?
 $EndSCHEMATC
